Commit message: changed the robot dimensions to fit actual and added pi

File: description/robot_core.xacro (robot description, xacro)
@@ -33,13 +33,13 @@
         <parent link="base_link"/>
         <child link="chassis"/>
-        <origin xyz="${-wheel_offset_x} 0 ${-wheel_offset_z}"/>
+        <origin xyz="${-wheel_offset_x} 0 ${wheel_offset_z}"/>
     </joint>
     <link name="chassis">
         <visual>
-            <origin xyz="${chassis_length/2} 0 ${chassis_height/2}"/>
+            <origin xyz="${chassis_length/2} 0 ${chassis_height/2}"/>         <!-- because object will always spwan with origin at the center-->
             <geometry>
                 <box size="${chassis_length} ${chassis_width} ${chassis_height}"/>
             </geometry>
-            <material name="orange"/>
+            <material name="white"/>
         </visual>
         <collision>
@@ -112,5 +112,5 @@
         <parent link="chassis"/>
         <child link="caster_wheel"/>
-        <origin xyz="${caster_wheel_offset_x} 0 ${caster_wheel_offset_z}"/>
+        <origin xyz="${caster_wheel_offset_x} 0 ${-caster_wheel_offset_z}"/>
     </joint>
     <link name="caster_wheel">
@@ -135,3 +135,25 @@
         <mu2 value="0.001"/>
     </gazebo>
+    <joint name="pi_joint" type="fixed">
+        <parent link="chassis"/>
+        <child link="pi_link"/>
+        <origin xyz="${pi_offset_x} 0 ${pi_offset_z}"/>
+    </joint>
+    <link name="pi_link">
+        <visual>
+            <geometry>
+                <box size="${pi_length} ${pi_width} ${pi_height}"/>
+            </geometry>
+            <material name="black"/>
+        </visual>
+        <collision>
+            <origin xyz="${pi_length/2} 0 ${pi_height/2}"/>
+            <geometry>
+                <box size="${pi_length} ${pi_width} ${pi_height}"/>
+            </geometry>
+        </collision>
+        <xacro:inertial_box mass="0.5" x="${pi_length}" y="${pi_width}" z="${pi_height}">
+            <origin xyz="${pi_offset_x} 0 ${pi_offset_z}" rpy="0 0 0"/>
+        </xacro:inertial_box>
+    </link>
 </robot>

File: description/robot_properties.xacro (robot description, xacro)
@@ -11,10 +11,17 @@
     <xacro:property name="wheel_mass" value="0.05"/>
     <xacro:property name="wheel_offset_x" value="0.055"/>
-    <xacro:property name="wheel_offset_y" value="0.0635"/>
-    <xacro:property name="wheel_offset_z" value="0.013"/>
+    <xacro:property name="wheel_offset_y" value="0.060"/>
+    <xacro:property name="wheel_offset_z" value="0.011"/>
 <!-- Castor Wheels-->
-    <xacro:property name="caster_wheel_radius" value="0.025"/>
+    <xacro:property name="caster_wheel_radius" value="0.02"/>
     <xacro:property name="caster_wheel_mass" value="0.01"/>
-    <xacro:property name="caster_wheel_offset_x" value="0.07"/>
-    <xacro:property name="caster_wheel_offset_z" value="0.04"/>
+    <xacro:property name="caster_wheel_offset_x" value="0.2"/>
+    <xacro:property name="caster_wheel_offset_z" value="0.02"/>
+<!-- Raspberry Pi-->
+    <xacro:property name="pi_length" value="0.095"/>
+    <xacro:property name="pi_width" value="0.065"/>
+    <xacro:property name="pi_height" value="0.03"/>
+    <xacro:property name="pi_mass" value="0.2"/>
+    <xacro:property name="pi_offset_x" value="0.2"/>
+    <xacro:property name="pi_offset_z" value="0.05"/>
 </robot>
